Commit message: add missing robot_footprint

File: src/my_robot/urdf/my_robot.xacro (robot description, xacro)
@@ -14,4 +14,10 @@
   </gazebo>
   <xacro:include filename="$(find my_robot)/urdf/my_robot.gazebo" />
+  <link name="robot_footprint"></link>
+  <joint name="robot_footprint_joint" type="fixed">
+    <origin xyz="0 0 0" rpy="0 0 0" />
+    <parent link="robot_footprint"/>
+    <child link="chassis" />
+  </joint>
   <link name='chassis'>
     <pose>0 0 0.15 0 0 0</pose>
